File: Eagle/Arduino/Arduino_S3v3_R2_b.brd (EAGLE design)
At the start: 84.8 x 67.3 mm, 43 parts, among them IC1 ATMEGA8 (OR 168), J1 PORT D(D0-D7), J2 PORT C(A0-A5), J3 PORT B(D8-D13), Q1 16000, T1 BC547, T2 BC557

Commit message: implemented gitview delete file - imroved eagle circiut for clock with measurement of current
Connections:
- net N$1 renamed D12
- net N$10 renamed D2
- net N$11 renamed D3
- net N$12 renamed D4
- net N$13 renamed D5
- net N$14 renamed D6
- net N$15 renamed D7
- net N$16 renamed A0
- net N$17 renamed A1
- net N$18 renamed A2
- net N$19 renamed A3
- net N$20 renamed A4
- net N$21 renamed A5
- net N$22 renamed D9
- net N$23 renamed D10
- net N$4 renamed D11
- net N$5 renamed D8

Commit message: Arduino-Eagle boards easyer basic design
Connections:
- net A4 renamed A4(SDA)
- net A5 renamed A5(SCL)
Changed lines of the file:
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@@
 <wire x1="35.56" y1="55.88" x2="35.56" y2="45.72" width="0.4064" layer="16"/>
 </signal>
-<signal name="A4">
+<signal name="A4(SDA)">
 <contactref element="IC1" pad="27"/>
 <contactref element="J2" pad="5"/>
 <wire x1="33.02" y1="55.88" x2="33.02" y2="45.72" width="0.4064" layer="16"/>
 </signal>
-<signal name="A5">
+<signal name="A5(SCL)">
 <contactref element="IC1" pad="28"/>
 <contactref element="J2" pad="6"/>
