File: Eagle/3LED-voltage-Level-Meter/VoltageLevelMeter3.brd (EAGLE design)
At the start: 31.4 x 34.3 mm, 14 parts, among them IC1 LM324N

Commit message: Renamed Names with spaces changed a circuit for voltage meter
Routing:
- net V+: track 32.3 -> 50.1 mm
- net N$6: track 12.7 -> 11.2 mm
- net N$1: track 38.7 -> 37.8 mm
Other:
- board size 31.4 x 34.3 mm -> 34 x 34.3 mm
Changed lines of the file:
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@@
 <board>
 <plain>
-<wire x1="33.02" y1="17.78" x2="64.44" y2="17.78" width="0" layer="20"/>
-<wire x1="64.44" y1="17.78" x2="64.44" y2="52.06" width="0" layer="20"/>
-<wire x1="64.44" y1="52.06" x2="33.02" y2="52.06" width="0" layer="20"/>
+<wire x1="33.02" y1="17.78" x2="66.98" y2="17.78" width="0" layer="20"/>
+<wire x1="66.98" y1="17.78" x2="66.98" y2="52.06" width="0" layer="20"/>
+<wire x1="66.98" y1="52.06" x2="33.02" y2="52.06" width="0" layer="20"/>
 <wire x1="33.02" y1="52.06" x2="33.02" y2="17.78" width="0" layer="20"/>
 <text x="35.56" y="53.34" size="1.778" layer="1" font="vector">1</text>
@@
 <text x="60.96" y="53.34" size="1.778" layer="1">11</text>
 <text x="63.5" y="53.34" size="1.778" layer="1">12</text>
-<text x="66.04" y="50.8" size="1.778" layer="1">1</text>
-<text x="66.04" y="48.26" size="1.778" layer="1">2</text>
-<text x="66.04" y="45.72" size="1.778" layer="1">3</text>
-<text x="66.04" y="43.18" size="1.778" layer="1">4</text>
-<text x="66.04" y="40.64" size="1.778" layer="1">5</text>
-<text x="66.04" y="38.1" size="1.778" layer="1">6</text>
-<text x="66.04" y="35.56" size="1.778" layer="1">7</text>
-<text x="66.04" y="33.02" size="1.778" layer="1">8</text>
-<text x="66.04" y="30.48" size="1.778" layer="1">9</text>
-<text x="66.04" y="27.94" size="1.778" layer="1">10</text>
-<text x="66.04" y="25.4" size="1.778" layer="1">11</text>
-<text x="66.04" y="22.86" size="1.778" layer="1">12</text>
-<text x="66.04" y="20.32" size="1.778" layer="1">13</text>
-<text x="66.04" y="17.78" size="1.778" layer="1">14</text>
-<text x="66.04" y="15.24" size="1.778" layer="1">15</text>
-<text x="66.04" y="12.7" size="1.778" layer="1">16</text>
+<text x="68.58" y="50.8" size="1.778" layer="1">1</text>
+<text x="68.58" y="48.26" size="1.778" layer="1">2</text>
+<text x="68.58" y="45.72" size="1.778" layer="1">3</text>
+<text x="68.58" y="43.18" size="1.778" layer="1">4</text>
+<text x="68.58" y="40.64" size="1.778" layer="1">5</text>
+<text x="68.58" y="38.1" size="1.778" layer="1">6</text>
+<text x="68.58" y="35.56" size="1.778" layer="1">7</text>
+<text x="68.58" y="33.02" size="1.778" layer="1">8</text>
+<text x="68.58" y="30.48" size="1.778" layer="1">9</text>
+<text x="68.58" y="27.94" size="1.778" layer="1">10</text>
+<text x="68.58" y="25.4" size="1.778" layer="1">11</text>
+<text x="68.58" y="22.86" size="1.778" layer="1">12</text>
+<text x="68.58" y="20.32" size="1.778" layer="1">13</text>
+<text x="68.58" y="17.78" size="1.778" layer="1">14</text>
+<text x="68.58" y="15.24" size="1.778" layer="1">15</text>
+<text x="68.58" y="12.7" size="1.778" layer="1">16</text>
 <wire x1="50.8" y1="38.608" x2="50.8" y2="37.592" width="0.1016" layer="145"/>
 <wire x1="50.292" y1="38.1" x2="51.308" y2="38.1" width="0.1016" layer="145"/>
@@
 <wire x1="52.07" y1="27.94" x2="52.07" y2="36.83" width="0.254" layer="1"/>
 <wire x1="52.07" y1="36.83" x2="50.8" y2="38.1" width="0.254" layer="1"/>
-<wire x1="48.26" y1="25.4" x2="48.26" y2="20.32" width="0.254" layer="16"/>
-<via x="48.26" y="20.32" extent="1-16" drill="0.6096"/>
+<wire x1="48.26" y1="20.32" x2="48.26" y2="25.4" width="0.254" layer="16"/>
+<via x="60.96" y="25.4" extent="1-16" drill="1"/>
+<wire x1="60.96" y1="25.4" x2="60.96" y2="20.32" width="0.254" layer="16"/>
+<wire x1="60.96" y1="20.32" x2="48.26" y2="20.32" width="0.254" layer="16"/>
 </signal>
 <signal name="N$1">
@@
 <contactref element="D1" pad="C"/>
 <wire x1="53.34" y1="43.18" x2="50.8" y2="43.18" width="0.4064" layer="16"/>
-<wire x1="53.34" y1="43.18" x2="60.96" y2="35.56" width="0.254" layer="16"/>
-<wire x1="60.96" y1="35.56" x2="60.96" y2="22.86" width="0.254" layer="16"/>
-<wire x1="60.96" y1="22.86" x2="53.34" y2="22.86" width="0.254" layer="16"/>
+<wire x1="53.34" y1="43.18" x2="63.5" y2="33.02" width="0.254" layer="16"/>
 <wire x1="53.34" y1="22.86" x2="53.34" y2="25.4" width="0.254" layer="16"/>
 <wire x1="50.8" y1="22.86" x2="53.34" y2="22.86" width="0.254" layer="16"/>
+<wire x1="63.5" y1="33.02" x2="63.5" y2="30.48" width="0.254" layer="16"/>
+<wire x1="55.88" y1="22.86" x2="53.34" y2="22.86" width="0.254" layer="16"/>
+<wire x1="63.5" y1="30.48" x2="55.88" y2="22.86" width="0.254" layer="16"/>
 </signal>
 <signal name="N$2">
@@
 <contactref element="IC1" pad="7"/>
 <contactref element="R7" pad="1"/>
-<wire x1="58.42" y1="35.56" x2="58.42" y2="25.4" width="0.4064" layer="16"/>
-<wire x1="55.88" y1="25.4" x2="58.42" y2="25.4" width="0.4064" layer="16"/>
+<wire x1="58.42" y1="35.56" x2="58.42" y2="27.94" width="0.4064" layer="16"/>
+<wire x1="55.88" y1="25.4" x2="58.42" y2="27.94" width="0.4064" layer="16"/>
 </signal>
 <signal name="N$7">
@@
 <wire x1="40.64" y1="45.72" x2="40.64" y2="43.18" width="0.4064" layer="16"/>
 </signal>
+<signal name="N$9">
+<via x="60.96" y="33.02" extent="1-16" drill="1"/>
+</signal>
+<signal name="N$13">
+<via x="66.04" y="33.02" extent="1-16" drill="1"/>
+</signal>
+<signal name="N$14">
+<via x="66.04" y="25.4" extent="1-16" drill="1"/>
+</signal>
 </signals>
