File: Eagle/Arduino/Projects/AlarmLeuchte/AlarmLeuchte.brd (EAGLE design)
At the start: 100 x 80 mm, 24 parts

Commit message: arduino switch on and off
Connections:
- removed net A2: S1.1, U$1.25
- net DIO2: now also S1.1, U$1.25
Routing:
- net DIO2: track 0.00 -> 12.1 mm
- net A2: track 4.48 -> 0.00 mm
Changed lines of the file:
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@@
 <setting verticaltext="up"/>
 </settings>
-<grid distance="0.1" unitdist="inch" unit="inch" style="lines" multiple="1" display="yes" altdistance="0.05" altunitdist="inch" altunit="inch"/>
+<grid distance="0.05" unitdist="inch" unit="inch" style="lines" multiple="1" display="yes" altdistance="0.05" altunitdist="inch" altunit="inch"/>
 <layers>
 <layer number="1" name="Top" color="4" fill="1" visible="yes" active="yes"/>
@@
 <signal name="DIO2">
 <contactref element="U$1" pad="4"/>
+<contactref element="S1" pad="1"/>
+<contactref element="U$1" pad="25"/>
+<wire x1="43.18" y1="43.18" x2="50.8" y2="43.18" width="0.254" layer="16"/>
+<wire x1="50.8" y1="43.18" x2="54.8894" y2="43.18" width="0.254" layer="16"/>
+<wire x1="54.8894" y1="43.18" x2="55.1688" y2="42.9006" width="0.254" layer="16"/>
 </signal>
 <signal name="DIO3(PWM)">
@@
 <wire x1="50.8" y1="45.72" x2="53.34" y2="45.72" width="0.508" layer="16"/>
 </signal>
-<signal name="A2">
-<contactref element="U$1" pad="25"/>
-<contactref element="S1" pad="1"/>
-<wire x1="50.8" y1="43.18" x2="54.8894" y2="43.18" width="0.254" layer="16"/>
-<wire x1="54.8894" y1="43.18" x2="55.1688" y2="42.9006" width="0.254" layer="16"/>
-</signal>
 <signal name="A1-SWITCH2">

Commit message: Alarmleuchte und pin controller mit timer funtion
Parts:
- added C3: (no value), rcl:E3,5-8
Connections:
- net GND: now also C3.-
- net VCC: now also C3.+
Routing:
- net GND: track 174.2 -> 175.5 mm
Changed lines of the file:
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@@
 <setting verticaltext="up"/>
 </settings>
-<grid distance="0.05" unitdist="inch" unit="inch" style="lines" multiple="1" display="yes" altdistance="0.05" altunitdist="inch" altunit="inch"/>
+<grid distance="0.1" unitdist="inch" unit="inch" style="lines" multiple="1" display="yes" altdistance="0.05" altunitdist="inch" altunit="inch"/>
 <layers>
 <layer number="1" name="Top" color="4" fill="1" visible="yes" active="yes"/>
@@
 <attribute name="VALUE" x="39.9542" y="21.336" size="1.27" layer="27" ratio="10" rot="R270"/>
 </element>
+<element name="C3" library="rcl" library_urn="urn:adsk.eagle:library:334" package="E3,5-8" package3d_urn="urn:adsk.eagle:package:23360/2" value="" x="32.163634375" y="53.34" smashed="yes">
+<attribute name="NAME" x="35.465634375" y="56.134" size="1.27" layer="25" ratio="10"/>
+<attribute name="POPULARITY" value="13" x="32.163634375" y="53.34" size="1.778" layer="27" display="off"/>
+<attribute name="SPICEPREFIX" value="C" x="32.163634375" y="53.34" size="1.778" layer="27" display="off"/>
+<attribute name="VALUE" x="29.877634375" y="50.292" size="1.27" layer="27" ratio="10"/>
+</element>
 </elements>
 <signals>
@@
 <wire x1="32.982625" y1="35.597375" x2="32.648025" y2="47.82910625" width="0.254" layer="16"/>
 <wire x1="32.982625" y1="35.597375" x2="33.02" y2="35.56" width="0.254" layer="16"/>
-<wire x1="32.648025" y1="47.82910625" x2="32.648025" y2="55.449740625" width="0.254" layer="16"/>
+<wire x1="32.648025" y1="47.82910625" x2="32.648025" y2="53.34" width="0.254" layer="16"/>
+<wire x1="32.648025" y1="53.34" x2="32.648025" y2="55.449740625" width="0.254" layer="16"/>
 <wire x1="32.667909375" y1="55.809071875" x2="32.648025" y2="55.449740625" width="0.254" layer="16"/>
 <wire x1="32.667909375" y1="55.809071875" x2="48.26" y2="55.809071875" width="0.254" layer="16"/>
@@
 <wire x1="48.401859375" y1="15.381859375" x2="48.26" y2="15.24" width="0.254" layer="16"/>
 <wire x1="33.02" y1="35.56" x2="30.48" y2="35.56" width="0.254" layer="16"/>
+<contactref element="C3" pad="-"/>
+<wire x1="33.941634375" y1="53.34" x2="32.648025" y2="53.34" width="0.254" layer="16"/>
 </signal>
 <signal name="X1">
@@
 <wire x1="43.18" y1="35.56" x2="40.64" y2="35.56" width="0.4064" layer="16"/>
 <wire x1="50.8" y1="30.48" x2="55.88" y2="30.48" width="0.254" layer="16"/>
+<contactref element="C3" pad="+"/>
+<wire x1="40.64" y1="35.56" x2="30.385634375" y2="53.34" width="0" layer="19" extent="1-1"/>
 </signal>
 <signal name="DIO5(PWM)">
